File: hardware/silice/Silice.kicad_sch (KiCad schematic)
At the start: 0 parts

Commit message: ACT3.7SLICEBackup
Parts:
- added EntradaP: USB4105-GF-A-060, USB4105-GF-A-060:GCT_USB4105-GF-A-060, symbol USB4105-GF-A-060:USB4105-GF-A-060
- added R1, R2: M55342K12B5E11RS2, Resistor_SMD:R_0201_0603Metric, symbol Device:R
- added U1: ESP32-S3-WROOM-1-N16R2, ESP32-S3-WROOM-1-N16R2:XCVR_ESP32-S3-WROOM-1-N16R2, symbol ESP32-S3-WROOM-1-N16R2:ESP32-S3-WROOM-1-N16R2
Connections:
- new net: EntradaP.A5 (CC1), R1.2
- new net: EntradaP.B5 (CC2), R2.2
- new net D_USBNegativo: EntradaP.A7 (DN1), EntradaP.B7 (DN2), U1.23 (IO21)
- new net D_USBPositivo: EntradaP.A6 (DP1), EntradaP.B6 (DP2), U1.14 (IO20)
- new net GND: EntradaP.A1_B12 (GND), EntradaP.B1_A12 (GND), EntradaP.SH1 (SHELL_GND), EntradaP.SH2 (SHELL_GND), EntradaP.SH3 (SHELL_GND), EntradaP.SH4 (SHELL_GND), R1.1, R2.1, U1.1 (GND), U1.40 (GND), U1.41_1 (GND), U1.41_2 (GND), U1.41_3 (GND), U1.41_4 (GND), U1.41_5 (GND), U1.41_6 (GND), U1.41_7 (GND), U1.41_8 (GND), U1.41_9 (GND)
- new net VBUS: EntradaP.A4_B9 (VBUS), EntradaP.B4_A9 (VBUS)

Commit message: AC1LSLICE
Parts:
- added U2: BQ25895RTW, Package_DFN_QFN:Texas_RTW_WQFN-24-1EP_4x4mm_P0.5mm_EP2.7x2.7mm_ThermalVias, symbol Battery_Management:BQ25895RTW
- added U3: TS3USB221ARSER, footprints:RSE10, symbol 2026-09-26_21-49-30:TS3USB221ARSER
- EntradaP: footprint USB4105-GF-A-060:GCT_USB4105-GF-A-060 -> GCT:GCT_USB4105-GF-A-060
Connections:
- net D_USBNegativo: now also U3.7 (D-); no longer U1.23 (IO21)
- net D_USBPositivo: now also U3.8 (D+); no longer U1.14 (IO20)
- net GND: now also U3.5 (GND), U3.6 (*OE)
- net VBUS: now also U2.1 (VBUS)
- net 2USB_N: now reaches U1.13 (IO19)
- net 2USB_N: now also U3.4 (2D-)
- new net: U2.13 (BAT), U2.14 (BAT)
- new net: U2.15 (SYS), U2.16 (SYS)
- new net: U2.17 (PGND), U2.18 (PGND), U2.25 (PGND)
- new net: U2.19 (SW), U2.20 (SW)
- new net 1USB_N: U2.3 (D-), U3.2 (1D-)
- new net 1USB_P: U2.2 (D+), U3.1 (1D+)
- new net 2USB_P: U1.14 (IO20), U3.3 (2D+)
Other:
- title: (none) -> SLICCE Proyect
